Commit message: update the URDF arm manipulator file

File: urdf_arm_manipulator/urdf/urdf_arm_manipulator.urdf (robot description, URDF)
Before this commit: robot urdf_arm_manipulator, 5 links, 4 joints
Links:
- link base_link: mass 0.11395 -> 0.99888
- link link_1: mass 0.11872 -> 0.18582
Joints:
- joint joint_1: axis 0 0 1 -> 0 1 0; origin xyz=0 0 0.0495 rpy=0 0 0 -> xyz=0 0 0.0465 rpy=1.5708 0 3.138
- joint joint_2: axis 0 1 0 -> 1 0 0; origin xyz=0 0 0.0255 rpy=0 0 0 -> xyz=0 0.0305 0 rpy=3.1416 0 -3.1416
- joint joint_3: axis 0 1 0 -> 1 0 0; origin xyz=0.0316 0 0.2992 rpy=0 0 0 -> xyz=0 0.2992 0.0316 rpy=0 0 0
- joint joint_4: axis 0 -1 0 -> 1 0 0; origin xyz=0.00185 0 0.2967 rpy=0 0 0 -> xyz=0 0.2967 0.00185 rpy=-1.5708 0 -3.1416
