Commit message: change pkg name urdf_manipulator>robot description

File: robot_description/urdf/urdf_manipulator.urdf (robot description, URDF)
Before this commit: robot urdf_manipulator, 6 links, 5 joints
Links:
- link base_link: geometry collision mesh filename=package://robot_description/meshes/base_link.STL; visual mesh filename=package://robot_description/meshes/base_link.STL
- link end_effector: geometry collision mesh filename=package://robot_description/meshes/end_effector.STL; visual mesh filename=package://robot_description/meshes/end_effector.STL
- link link_1: geometry collision mesh filename=package://robot_description/meshes/link_1.STL; visual mesh filename=package://robot_description/meshes/link_1.STL
- link link_2: geometry collision mesh filename=package://robot_description/meshes/link_2.STL; visual mesh filename=package://robot_description/meshes/link_2.STL
- link link_3: geometry collision mesh filename=package://robot_description/meshes/link_3.STL; visual mesh filename=package://robot_description/meshes/link_3.STL
- link link_4: geometry collision mesh filename=package://robot_description/meshes/link_4.STL; visual mesh filename=package://robot_description/meshes/link_4.STL
